File: TSOC_USBUART2/revisions/TSOC_USBUART2.brd (EAGLE design)
At the start: 45.7 x 25.4 mm, 41 parts, among them J1 JMP-3-1_2, J2 JMP-3-1_2, P1 M08, P1A M08PTH, U1 MIC5219 3.3V, U2 CY7C65215-32-PROTO

Commit message: update to Rev1.0
Parts:
- moved C2 6.48 mm to (31.5, 21.6)
- moved C7 6.48 mm to (22.9, 18.0)
- moved C8 6.48 mm to (22.4, 10.7)
- moved FID1 6.48 mm to (1.27, 24.1)
- moved FID4 6.48 mm to (40.6, 24.1)
- moved P1 6.48 mm to (42.2, 12.7)
- moved P1A 6.48 mm to (43.2, 21.6)
- moved R13 6.48 mm to (31.0, 17.5)
- moved R4 6.48 mm to (5.08, 21.6)
- moved SUSPEND 6.48 mm to (2.03, 21.6)
- moved TSOC 6.48 mm to (16.5, 12.7)
- moved U$1 6.48 mm to (19.1, 12.7)
- moved USB 6.48 mm to (2.03, 12.7)
- moved C1 6.48 mm to (8.64, 7.87)
- moved C3 6.48 mm to (31.5, 3.56)
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