File: TSOC_USBUART2/revisions/TSOC_USBUART2_R3_0.brd (EAGLE design)
At the start: 50.8 x 30.5 mm, 42 parts, among them J1 JMP-3-1_2, J2 JMP-3-1_2, U1 MIC5219 3.3V, U2 CY7C65215-32-PROTO

Commit message: update to V4_0
Parts:
- removed FUSE: 500mA-PTC, SparkFun:PTC-1206
- removed J3: (no value), PatternAgents-ProtoPads:2X8
- removed U$8: TSOC-LOGO-SMALL, thingSoC:TSOC-LOGO-SML
- added F1: 1A, TSOC_USBUART2:EIA-0603
- added P1: M08, TSOC_USBUART2:1X08-SMD-FEMALE
- added P1A: M08PTH, TSOC_USBUART2:1X08
- moved U$1 23.9 mm to (14.9, 5.97)
Connections:
- net !CTS1: now also P1.7, P1A.7; no longer J3.14
- net !DSR1: now also P1.1, P1A.1; no longer J3.2
- net !DTR1: now also P1.3, P1A.3; no longer J3.6
- net !RTS1: now also P1.2, P1A.2; no longer J3.4
- net 5V0: now also F1.1; no longer FUSE.2
- net GND: now also P1.8, P1A.8; no longer J3.15, J3.16
- net RXD1: now also P1.4, P1A.4; no longer J3.10
- net TXD1: now also P1.5, P1A.5; no longer J3.8
- net USB1_VBUS: now also F1.2; no longer FUSE.1
- net VCC: now also P1.6, P1A.6; no longer J3.11, J3.12
Routing:
- net RXD1: track 37.8 -> 44.6 mm, vias 3 -> 5
- net TXD1: track 42.8 -> 47.1 mm
- net !CTS1: track 44.4 -> 48.2 mm
- net !RTS1: track 63.3 -> 66.9 mm
- net GND: track 166.8 -> 164.2 mm
- net VCC: track 111.2 -> 109.6 mm
- net USB1_VBUS: track 22.3 -> 21.1 mm
- net 5V0: track 52.2 -> 51.2 mm
Other:
- board text added: "Rev. 3.0"
- board text removed: "@PatternAgents"
- board text removed: "Pattern Agents"
- board text removed: "Rev. 4.0"
