File: TSOC_USBUART2/revisions/TSOC_USBUART2_R3_0.sch (EAGLE design)
At the start: 41 parts, among them J1 JMP-3-1_2, J2 JMP-3-1_2, U1 MIC5219 3.3V, U2 CY7C65215-32-PROTO

Commit message: update to V4_0
Parts:
- removed FUSE: 500mA-PTC, SparkFun:PTCSMD
- removed J3: (no value), PatternAgents-ProtoPads:M08X2
- removed U$8: TSOC-LOGO-SMALL, thingSoC:TSOC-LOGO-SMALL
- added F1: 1A, TSOC_USBUART2:FUSE
- added P1: M08, TSOC_USBUART2:M08
- added P1A: M08PTH, TSOC_USBUART2:M08PTH
- added U$1: TSOC-LOGO-SMALL, thingSoC:TSOC-LOGO-SMALL
Connections:
- net !CTS1: now also P1.7, P1A.7; no longer J3.14
- net !DSR1: now also P1.1, P1A.1; no longer J3.2
- net !DTR1: now also P1.3, P1A.3; no longer J3.6
- net !RTS1: now also P1.2, P1A.2; no longer J3.4
- net 5V0: now also F1.P$1; no longer FUSE.2
- net GND: now also P1.8, P1A.8; no longer J3.15, J3.16
- net RXD1: now also P1.4, P1A.4; no longer J3.10
- net TXD1: now also P1.5, P1A.5; no longer J3.8
- net USB1_VBUS: now also F1.P$2; no longer FUSE.1
- net VCC: now also P1.6, P1A.6; no longer J3.11, J3.12
Other:
- note added: "PPTC Fuse (0603)"
- note removed: "!CTS"
- note removed: "!DEBUG"
- note removed: "!DTR"
- note removed: "!RESET"
- note removed: "!RTS"
- note removed: "GROUND"
- note removed: "I2C-SDA"
- note removed: "I2C-SDL"
- note removed: "POWER"
- note removed: "RXD"
- note removed: "SWDCLK"
- note removed: "SWDIO"
- note removed: "TXD"
