File: TSOC_USBUART2/TSOC_USBUART2.brd (EAGLE design)
At the start: 50.8 x 30.5 mm, 41 parts, among them J1 JMP-3-1_2, J2 JMP-3-1_2, P1 M08, P1A M08PTH, U1 MIC5219 3.3V, U2 CY7C65215-32-PROTO

Commit message: update to Rev2.0
Parts:
- moved FID3 4.54 mm to (39.9, 1.78)
- moved FID4 4.54 mm to (39.9, 28.7)
- moved FID1 0.51 mm to (4.57, 28.7)
- moved FID2 0.36 mm to (4.57, 1.78)
- moved U$4 0.36 mm to (4.57, 1.78)
- moved U$5 0.36 mm to (4.57, 1.78)
- moved U$6 0.36 mm to (4.57, 1.78)
Routing:
- net GND: track 162.1 -> 164.2 mm
Changed lines of the file:
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@@
 <grid distance="10" unitdist="mil" unit="mil" style="lines" multiple="1" display="yes" altdistance="10" altunitdist="mil" altunit="mil"/>
 <layers>
-<layer number="1" name="Top" color="4" fill="1" visible="no" active="yes"/>
+<layer number="1" name="Top" color="4" fill="1" visible="yes" active="yes"/>
 <layer number="2" name="Route2" color="1" fill="3" visible="no" active="no"/>
 <layer number="3" name="Route3" color="4" fill="3" visible="no" active="no"/>
@@
 <layer number="19" name="Unrouted" color="6" fill="1" visible="yes" active="yes"/>
 <layer number="20" name="Dimension" color="15" fill="1" visible="yes" active="yes"/>
-<layer number="21" name="tPlace" color="7" fill="1" visible="no" active="yes"/>
+<layer number="21" name="tPlace" color="7" fill="1" visible="yes" active="yes"/>
 <layer number="22" name="bPlace" color="7" fill="1" visible="yes" active="yes"/>
 <layer number="23" name="tOrigins" color="15" fill="1" visible="yes" active="yes"/>
 <layer number="24" name="bOrigins" color="15" fill="1" visible="yes" active="yes"/>
-<layer number="25" name="tNames" color="7" fill="1" visible="yes" active="yes"/>
+<layer number="25" name="tNames" color="7" fill="1" visible="no" active="yes"/>
 <layer number="26" name="bNames" color="7" fill="1" visible="no" active="yes"/>
 <layer number="27" name="tValues" color="7" fill="1" visible="no" active="yes"/>
@@
 <attribute name="VALUE" x="34.671" y="16.6878" size="0.4064" layer="27" rot="R90"/>
 </element>
-<element name="FID2" library="TSOC-ESP8266-BASE" package="MICRO-FIDUCIAL" value="FIDUCIALUFIDUCIAL" x="4.318" y="1.524"/>
-<element name="FID3" library="TSOC-ESP8266-BASE" package="MICRO-FIDUCIAL" value="FIDUCIALUFIDUCIAL" x="43.942" y="3.81"/>
-<element name="FID4" library="TSOC-ESP8266-BASE" package="MICRO-FIDUCIAL" value="FIDUCIALUFIDUCIAL" x="43.942" y="26.67" smashed="yes"/>
-<element name="FID1" library="TSOC-ESP8266-BASE" package="MICRO-FIDUCIAL" value="FIDUCIALUFIDUCIAL" x="4.064" y="28.702"/>
+<element name="FID2" library="TSOC-ESP8266-BASE" package="MICRO-FIDUCIAL" value="FIDUCIALUFIDUCIAL" x="4.572" y="1.778"/>
+<element name="FID3" library="TSOC-ESP8266-BASE" package="MICRO-FIDUCIAL" value="FIDUCIALUFIDUCIAL" x="39.878" y="1.778"/>
+<element name="FID4" library="TSOC-ESP8266-BASE" package="MICRO-FIDUCIAL" value="FIDUCIALUFIDUCIAL" x="39.878" y="28.702" smashed="yes"/>
+<element name="FID1" library="TSOC-ESP8266-BASE" package="MICRO-FIDUCIAL" value="FIDUCIALUFIDUCIAL" x="4.572" y="28.702"/>
 <element name="TSOC" library="thingSoC" package="TSOC-BB-S32" value="TSOC-32-BB" x="19.812" y="15.24" smashed="yes"/>
 <element name="POWER" library="TSOC-ESP8266-BASE" package="LED-0603" value="GRN" x="2.286" y="21.59" smashed="yes" rot="R90">
@@
 </element>
 <element name="U$3" library="thingSoC" package="TSOC-LOGO-LRG" value="TSOC-LOGO-LRG" x="33.02" y="17.018" rot="MR0"/>
-<element name="U$4" library="thingSoC" package="TSOC-LOGO-BLANK" value="TSOC-LOGO" x="4.318" y="1.524"/>
-<element name="U$5" library="thingSoC" package="TSOC-LOGO-BLANK" value="TSOC-LOGO" x="4.318" y="1.524"/>
-<element name="U$6" library="thingSoC" package="TSOC-LOGO-BLANK" value="TSOC-LOGO" x="4.318" y="1.524"/>
+<element name="U$4" library="thingSoC" package="TSOC-LOGO-BLANK" value="TSOC-LOGO" x="4.572" y="1.778"/>
+<element name="U$5" library="thingSoC" package="TSOC-LOGO-BLANK" value="TSOC-LOGO" x="4.572" y="1.778"/>
+<element name="U$6" library="thingSoC" package="TSOC-LOGO-BLANK" value="TSOC-LOGO" x="4.572" y="1.778"/>
 <element name="C2" library="TSOC_USBUART2" package="EIA-1206" value="22uF" x="34.798" y="24.13" smashed="yes">
 <attribute name="NAME" x="32.131" y="23.622" size="0.6096" layer="25" font="vector" ratio="15" rot="R90"/>
@@
 <signal name="GND" class="1">
 <polygon width="0.254" layer="1" spacing="0.254" pour="hatch" isolate="0.254" orphans="yes">
-<vertex x="47.752" y="27.94"/>
-<vertex x="47.752" y="2.54"/>
-<vertex x="9.652" y="2.54"/>
-<vertex x="9.652" y="27.94"/>
+<vertex x="44.196" y="28.956"/>
+<vertex x="44.196" y="1.524"/>
+<vertex x="9.652" y="1.524"/>
+<vertex x="9.652" y="28.956"/>
 </polygon>
 <polygon width="0.254" layer="16" spacing="0.254" pour="hatch" isolate="0.254" orphans="yes">
-<vertex x="47.752" y="27.94"/>
-<vertex x="47.752" y="2.54"/>
-<vertex x="9.652" y="2.54"/>
-<vertex x="9.652" y="27.94"/>
+<vertex x="44.196" y="28.956"/>
+<vertex x="44.196" y="1.524"/>
+<vertex x="9.652" y="1.524"/>
+<vertex x="9.652" y="28.956"/>
 </polygon>
 <contactref element="C1" pad="2"/>
@@
 <wire x1="25.582" y1="8.128" x2="25.582" y2="10.016" width="0.6096" layer="1"/>
 <wire x1="25.582" y1="10.016" x2="25.654" y2="9.868" width="0.6096" layer="1"/>
-<wire x1="37.338" y1="7.236" x2="37.338" y2="13.208" width="0.6096" layer="1"/>
+<wire x1="37.338" y1="7.236" x2="37.338" y2="7.62" width="0.6096" layer="1"/>
+<wire x1="37.338" y1="7.62" x2="37.338" y2="13.208" width="0.6096" layer="1"/>
 <wire x1="36.83" y1="21.844" x2="37.338" y2="22.352" width="0.6096" layer="16"/>
 <wire x1="11.176" y1="21.8948" x2="12.6492" y2="21.8948" width="0.6096" layer="1"/>
@@
 <wire x1="36.322" y1="22.352" x2="36.322" y2="24.006" width="0.6096" layer="1"/>
 <wire x1="36.322" y1="24.006" x2="36.198" y2="24.13" width="0.6096" layer="1"/>
-<wire x1="36.198" y1="6.096" x2="36.198" y2="3.934" width="0.8128" layer="1"/>
+<wire x1="36.198" y1="6.096" x2="36.198" y2="5.1562" width="0.8128" layer="1"/>
+<wire x1="36.198" y1="5.1562" x2="36.198" y2="4.8006" width="0.8128" layer="1"/>
+<wire x1="36.198" y1="4.8006" x2="36.198" y2="3.934" width="0.8128" layer="1"/>
 <wire x1="36.198" y1="3.934" x2="36.322" y2="3.81" width="0.8128" layer="1"/>
 <wire x1="37.338" y1="7.236" x2="36.198" y2="6.096" width="0.6096" layer="1"/>
@@
 <wire x1="4.882" y1="13.152" x2="5.08" y2="12.954" width="0.4064" layer="1"/>
 <wire x1="5.08" y1="12.954" x2="9.144" y2="12.954" width="0.4064" layer="1"/>
-<wire x1="46.7614" y1="6.4008" x2="46.482" y2="6.35" width="0.254" layer="16"/>
-<wire x1="47.4726" y1="5.6896" x2="47.51710625" y2="5.6572625" width="0.254" layer="16"/>
-<wire x1="47.117" y1="6.4008" x2="46.482" y2="6.35" width="0.254" layer="16"/>
-<wire x1="46.9392" y1="6.4008" x2="46.482" y2="6.35" width="0.254" layer="16"/>
 <wire x1="36.2712" y1="5.5118" x2="36.198" y2="6.096" width="0.254" layer="1"/>
 <wire x1="36.0934" y1="6.0452" x2="36.198" y2="6.096" width="0.254" layer="1"/>
 <wire x1="36.0934" y1="6.0452" x2="36.071003125" y2="5.9689875" width="0.254" layer="1"/>
-<wire x1="36.0934" y1="4.0894" x2="36.322" y2="3.81" width="0.254" layer="1"/>
-<wire x1="36.0934" y1="4.0894" x2="36.195" y2="4.0894" width="0.254" layer="1"/>
 <wire x1="36.2712" y1="6.0452" x2="36.198" y2="6.096" width="0.254" layer="1"/>
 <wire x1="36.2712" y1="6.0452" x2="36.2712" y2="5.9689875" width="0.254" layer="1"/>
 <wire x1="36.2712" y1="5.6896" x2="36.198" y2="6.096" width="0.254" layer="1"/>
 <wire x1="36.2712" y1="5.8674" x2="36.198" y2="6.096" width="0.254" layer="1"/>
-<wire x1="47.117" y1="6.4008" x2="47.4726" y2="5.6896" width="0" layer="19" extent="16-16"/>
+<wire x1="36.6268" y1="4.2672" x2="36.6268" y2="5.8674" width="0.254" layer="1"/>
+<wire x1="36.449" y1="4.0894" x2="36.6268" y2="4.2672" width="0.254" layer="1"/>
+<wire x1="36.449" y1="4.2672" x2="36.322" y2="3.81" width="0.254" layer="1"/>
+<wire x1="36.449" y1="4.2672" x2="36.44899375" y2="4.2672" width="0.254" layer="1"/>
+<wire x1="36.449" y1="4.0894" x2="36.322" y2="3.81" width="0.254" layer="1"/>
+<wire x1="36.449" y1="4.0894" x2="36.44899375" y2="4.0894" width="0.254" layer="1"/>
+<wire x1="37.3634" y1="7.6454" x2="37.338" y2="7.62" width="0.254" layer="1"/>
+<wire x1="36.0934" y1="5.1562" x2="36.198" y2="5.1562" width="0.254" layer="1"/>
+<wire x1="36.2712" y1="4.8006" x2="36.198" y2="4.8006" width="0.254" layer="1"/>
+<wire x1="36.2712" y1="4.0894" x2="36.322" y2="3.81" width="0.254" layer="1"/>
+<wire x1="36.0934" y1="4.0894" x2="36.322" y2="3.81" width="0.254" layer="1"/>
+<wire x1="36.0934" y1="4.0894" x2="36.195" y2="4.0894" width="0.254" layer="1"/>
+<wire x1="28.2702" y1="10.3124" x2="28.2702" y2="10.32885625" width="0.254" layer="1"/>
+<wire x1="27.9146" y1="9.4234" x2="27.94" y2="9.4281" width="0.254" layer="1"/>
+<wire x1="27.9146" y1="9.4234" x2="27.9505" y2="9.43861875" width="0.254" layer="1"/>
+<wire x1="27.9146" y1="9.6012" x2="27.94" y2="9.4281" width="0.254" layer="1"/>
+<wire x1="27.9146" y1="9.6012" x2="27.9505" y2="9.6012" width="0.254" layer="1"/>
+<wire x1="27.9146" y1="10.3124" x2="27.9505" y2="10.332896875" width="0.254" layer="1"/>
 </signal>
 <signal name="5V0">
