File: TSOC_USBUART2/revisions/R5_1/TSOC_USBUART2_pwr.sch (EAGLE design)
At the start: 41 parts, among them J1 JMP-3-1_2, J2 JMP-3-1_2, U1 CY7C65215-32-PROTO, U2 MIC5219 3.3V

Commit message: update to Rev5.0
Parts:
- removed $$U$2, U$3: TSOC-LOGO, thingSoC:TSOC-LOGO
- removed DPC: (no value), PatternAgents-ProtoPads:M08X2
- removed FUSE: 500mA-PTC, SparkFun:PTCSMD
- removed J1, J2: JMP-3-1_2, PatternAgents-ProtoPads:JMP-3-1_2
- removed PORT1: YELLOW, TSOC-ESP8266-BASE:LED0603
- removed PORT2: BLUE, TSOC-ESP8266-BASE:LED0603
- removed POWER: GRN, TSOC-ESP8266-BASE:LED0603
- removed R4: 1K, TSOC_USBUART2:RESISTOR-0603
- removed R7: 22, TSOC_USBUART2:RESISTOR-0603
- removed SUSPEND: RED, TSOC-ESP8266-BASE:LED0603
- removed TSOC: TSOC-24-BB, thingSoC:TSOC-24-BB
- removed U$4: TSOC-PCB-SINGLE, thingSoC:TSOC-PCB-SINGLE
- removed U$6: TSOC-LOGO-SMALL, thingSoC:TSOC-LOGO-SMALL
- added A: TSOC-24-BB, thingSoC:TSOC-24-BB
- added BATTERY: (no value), TSOC-ESP8266-BASE:JST_2MM_MALE
- added C10, C16, C9: 100nf, Seeed-Capacitor-2016:CERAMIC-100NF-50V-10%-X7R(0603)
- added C17: 47uf, Seeed-Capacitor-2016:TANTALUM-SMD-47UF-6.3V(AVX-A)
- added D2: 20V-1A, Seeed-Diode-2016:SMD-DIODE-SCHOTTKY-20V-1A(SOD-123)
- added F1: 500mA-PTC, SparkFun:PTCSMD
- added J1P: (no value), TSOC-ESP8266-BASE:M02-JST-2-PTH-NO_SILK
- added J3: (no value), PatternAgents-ProtoPads:M08X2
- added L1: 330OHM-500MA, Seeed-Inductor-2016:SMD-FERRITE-CHIP-120-OHM-500MA(0603)
- added LED1: GREEN-0603, Seeed-LED-2016:SMD-LED-CLEAR-GREEN(0603)
- added LED2: YELLOW-0603, Seeed-LED-2016:SMD-LED-CLEAR-YELLOW(0603)
- added R11: 10K 1/10W, Seeed-Resistor-2016:SMD-RES-10K-5%-1/10W(0603)
- added R13: 22K, Seeed-Resistor-2016:SMD-RES-22K-5%-1/10W(0603)
- added R15: 10K, Seeed-Resistor-2016:SMD-RES-10K-1%-1/10W(0603)
- added RESET, USER: B3U-1000P-2P-SMD, Seeed-Switch-2016:SMD-BUTTON(2P-3.0X2.5X1.2+0.4MM)-B3U-1000P-2P-SMD
- added U$101: TSOC-LOGO-SMALL, thingSoC:TSOC-LOGO-SMALL
- added U3: CY7C65215-32-PROTO, PatternAgents-Cypress:CY7C65215-32-PROTO
- added VCC: JMP-3-1_2, PatternAgents-ProtoPads:JMP-3-1_2
- C1, C4: value 470pF -> 100nf; device TSOC_USBUART2:CAP-0603 -> Seeed-Capacitor-2016:CERAMIC-100NF-50V-10%-X7R(0603)
- C2: value 1.0uF -> 1uf; device TSOC_USBUART2:CAP-0603 -> Seeed-Capacitor-2016:CERAMIC-1UF-25V-10%-X7R(0603)
- C3, C5: value 0.1uF -> 10uf; device TSOC_USBUART2:CAP-0603 -> Seeed-Capacitor-2016:CERAMIC-10UF-10V-10%-X5R(0603)
- C6: value 0.1uF -> 1uf; device TSOC_USBUART2:CAP-0603 -> Seeed-Capacitor-2016:CERAMIC-1UF-25V-10%-X7R(0603)
- C7: value 22uF -> 10uf; device TSOC_USBUART2:CAP-1206 -> Seeed-Capacitor-2016:CERAMIC-10UF-10V-10%-X5R(0603)
- C8: value 22uF -> 1uf; device TSOC_USBUART2:CAP-1206 -> Seeed-Capacitor-2016:CERAMIC-1UF-25V-10%-X7R(0603)
- D1: value 5V-225MW -> 20V-1A; device Seeed-Diode-2016:SMD-DIODE-TVS-5V-225MW(SOT-23) -> Seeed-Diode-2016:SMD-DIODE-SCHOTTKY-20V-1A(SOD-123)
- R1, R2: value 1K -> 1K 1/10W; device TSOC_USBUART2:RESISTOR-0603 -> Seeed-Resistor-2016:SMD-RES-1K-5%-1/10W(0603)
- R10: value 22K -> 10K 1/10W; device TSOC_USBUART2:RESISTOR-0603 -> Seeed-Resistor-2016:SMD-RES-10K-5%-1/10W(0603)
- R3: value 1K -> 1M 1/10W; device TSOC_USBUART2:RESISTOR-0603 -> Seeed-Resistor-2016:SMD-RES-1M-5%-1/10W(0603)
- R5: value 1M -> 22R; device TSOC_USBUART2:RESISTOR-0603 -> Seeed-Resistor-2016:SMD-RES-22R-5%-1/10W(0603)
- R6: value 22 -> 22R; device TSOC_USBUART2:RESISTOR-0603 -> Seeed-Resistor-2016:SMD-RES-22R-5%-1/10W(0603)
- R8, R9: value 10K -> 10K 1/10W; device TSOC_USBUART2:RESISTOR-0603 -> Seeed-Resistor-2016:SMD-RES-10K-5%-1/10W(0603)
- U$1: value TSOC-LOGO -> TSOC-PCB-SINGLE; device thingSoC:TSOC-LOGO -> thingSoC:TSOC-PCB-SINGLE
- U1: value CY7C65215-32-PROTO -> AP2112K-3.3V; device PatternAgents-Cypress:CY7C65215-32-PROTO -> SparkFun-PowerIC:V_REG_LDOSMD; PROD_ID (none) -> VREG-12457
- U2: value MIC5219 3.3V -> MCP73831; device TSOC-ESP8266-BASE:V_REG_MIC52193.3V -> TSOC-ESP8266-BASE:MCP73831
Connections:
- removed net !USB_RST: R8.2, U1.!XRES
- removed net BLU: PORT2.A, R2.1
- removed net GRN: POWER.A, R3.1
- removed net RED: R4.1, SUSPEND.A
- removed net TXDEN_0: J1.3, U1.GPIO17
- removed net USB1_ID: USB.USBID
- removed net USB1_VBUS: FUSE.1, USB.VBUS
- removed net YEL: PORT1.A, R1.1
- new net !XRES: C16.1, R11.1, RESET.2, U3.!XRES
- new net CLED: LED2.-, R2.2
- new net CSTAT: R2.1, U2.STAT
- new net DCD: U3.GPIO16
- new net N$17: LED1.+, R1.1
- new net SCL: A.SCL, J3.3, R9.1
- new net SDA: A.SDA, J3.13, R10.1
- new net VBAT: BATTERY.+, C2.1, D2.+, J1P.1, U2.VBAT
- new net VBUS: C6.1, D1.+, LED2.+, R13.1, U2.VIN, U3.VBUS@19, USB.VBUS
- new net VDDIO: C10.2, C9.2, L1.2, R1.2, R10.2, R11.2, R9.2, U3.VDDD@1, U3.VDDD@23
- new net VIN: D1.-, D2.-, F1.1
- new net WAKE: U3.WAKEUP, USER.2
- net !CTS: now also A.!CTS, U3.GPIO4; no longer TSOC.!CTS, U1.GPIO4
- net !CTS1: now also J3.14, U3.GPIO13; no longer DPC.14, U1.GPIO13
- net !DCD: now also A.!DCD; no longer TSOC.!DCD, U1.GPIO16
- net !DSR: now also A.!DSR, U3.GPIO2; no longer TSOC.!DSR, U1.GPIO2
- net !DSR1: now also J3.2, U3.GPIO14; no longer DPC.2, U1.GPIO14
- net !DTR: now also A.!DTR, U3.GPIO9; no longer TSOC.!DTR, U1.GPIO9
- net !DTR1: now also J3.6, U3.GPIO15; no longer DPC.6, U1.GPIO15
- net !POWER: now also LED1.-, U3.GPIO6; no longer POWER.C, U1.GPIO6
- net !RI: now also A.!RI, U3.GPIO17; no longer TSOC.!RI, U1.WAKEUP
- net !RTS: now also A.!RTS, U3.GPIO3; no longer J1.1, U1.GPIO3
- net !RTS1: now also J3.4, U3.GPIO12; no longer DPC.4, U1.GPIO12
- net !RX_LED: now also U3.GPIO1; no longer PORT1.C, U1.GPIO1
- net !TX_LED: now also U3.GPIO0; no longer PORT2.C, U1.GPIO0
- net 3V3: now also A.3V3, C3.2, U1.OUT, VCC.1; no longer C7.1, J2.1, TSOC.3V3, U2.OUT
- net 5V0: now also A.5V0, C5.1, F1.2, J3.12, U1.EN, U1.IN, VCC.3; no longer C3.1, C8.1, DPC.12, FUSE.2, J2.3, R10.1, TSOC.5V0, U1.VBUS@19, U2.EN, U2.IN
- net BUS_DET: now also R13.2, R15.1, U3.GPIO7; no longer R10.2, R9.1, U1.GPIO7
- net BYPASS1: now also U1.BP; no longer U2.BP
- net GND: now also A.AGND, A.GND, BATTERY.-, C10.1, C16.2, C17.-, C2.2, C3.1, C5.2, C6.2, C7.1, C8.1, C9.1, J1P.2, J3.15, J3.16, R15.2, R3.2, R8.1, RESET.1, U1.GND, U2.VSS, U3.VSSA@24, U3.VSSD@17, U3.VSSD@20, U3.VSSD@4, USER.1; no longer C2.1, C3.2, C5.1, C6.1, C7.2, C8.2, D1.3, DPC.15, DPC.16, R5.2, R9.2, TSOC.AGND, TSOC.GND, U1.VSSA@24, U1.VSSD@17, U1.VSSD@20, U1.VSSD@4, U2.GND
- net N$1: now also R8.2, U2.PROG; no longer J1.2, TSOC.!RTS
- net RXD: now also A.RXD, U3.GPIO8; no longer TSOC.RXD, U1.GPIO8
- net RXD1: now also J3.8, U3.GPIO10; no longer DPC.8, U1.GPIO10
- net SUSP: now also U3.SUSPEND; no longer SUSPEND.C, U1.SUSPEND
- net TXD: now also A.TXD, U3.GPIO5; no longer TSOC.TXD, U1.GPIO5
- net TXD1: now also J3.10, U3.GPIO11; no longer DPC.10, U1.GPIO11
- net TXDEN_1: now also J3.1, U3.GPIO18; no longer DPC.1, U1.GPIO18
- net USB1_DM: now also R6.2, U3.USBDM; no longer D1.2, R6.1, USB.D-
- net USB1_DP: now also R5.2, U3.USBDP; no longer D1.1, R7.1, USB.D+
- net USB1_M: now also R6.1, USB.D-; no longer R6.2, U1.USBDM
- net USB1_P: now also R5.1, USB.D+; no longer R7.2, U1.USBDP
- net USB1_SHIELD: now also R3.1; no longer R5.1
- net VCC: now also C17.+, C7.2, J3.11, L1.1, VCC.2; no longer C5.2, C6.2, DPC.11, J2.2, R1.2, R2.2, R3.2, R4.2, R8.1, U1.VDDD@1, U1.VDDD@23
- net VCCD1: now also C8.2, U3.VCCD@16; no longer C2.2, U1.VCCD@16
Other:
- note added: "I/O Voltage Level Selection and Input Power Filtering"
- note added: "I2C Pullups"
- note added: "I2C-SCL"
- note added: "Li-Po Battery Charger"
- note added: "Reset Pullup"
- note added: "Switches"
- note added: "USB Power and Interface"
- note added: "USB_ENUM LED"
- note added: "thingSoC DPC Digital Programming Connector"
- note removed: "I2C-SDL"
- note removed: "thingSoC Module Template"
- note removed: "thingSoC USBUART2 "Base" Reference Design Page A : thingSoC IoT Socket Page B : 3.3 Volt Power Supply Page C : Dual USB to UART Bridge Device Page D : USB-UART Output Connector"
