File: TSOC_USBUART2/revisions/R5_1/TSOC_USBUART2_R5_1.brd (EAGLE design)
At the start: 44.5 x 30.5 mm, 43 parts, among them J1 JMP-3-1_2, J2 JMP-3-1_2, U1 CY7C65215-32-PROTO, U2 AP2112K-3.3V

Commit message: update R5
Parts:
- renumbered PORT2 to DPC
Changed lines of the file:
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@@
 </element>
 <element name="C3" library="Seeed-Capacitor-2016" package="C0603" value="100nf" x="24.003" y="11.176" smashed="yes" rot="R90">
-<attribute name="NAME" x="22.479" y="10.668" size="0.8128" layer="25" font="vector" ratio="15" rot="R180"/>
+<attribute name="NAME" x="24.892" y="10.287" size="0.8128" layer="25" font="vector" ratio="15" rot="R180"/>
 <attribute name="VALUE" value="100nf" x="23.749" y="9.906" size="0.4064" layer="27" rot="R270"/>
 <attribute name="MPN" value="CC0603KRX7R9BB104" x="24.003" y="11.176" size="1.778" layer="27" rot="R90" display="off"/>
@@
 <element name="U$4" library="thingSoC" package="TSOC-BB-BRD-DIM" value="TSOC-PCB-SINGLE" x="18.796" y="15.24" rot="R90"/>
 <element name="U$5" library="thingSoC" package="TSOC-LOGO-SML" value="TSOC-LOGO-SMALL" x="37.592" y="2.794"/>
-<element name="PORT2" library="PatternAgents-ProtoPads" package="2X8" value="" x="42.545" y="24.13" smashed="yes" rot="MR270">
+<element name="DPC" library="PatternAgents-ProtoPads" package="2X8" value="" x="42.545" y="24.13" smashed="yes" rot="MR270">
 <attribute name="VALUE" x="45.72" y="25.4" size="1.27" layer="28" rot="MR270"/>
 </element>
@@
 <wire x1="36.3474" y1="7.6454" x2="36.322" y2="7.62" width="0.254" layer="1"/>
 <wire x1="26.8986" y1="9.6012" x2="26.9345" y2="9.6012" width="0.254" layer="1"/>
-<contactref element="PORT2" pad="15"/>
-<contactref element="PORT2" pad="16"/>
+<contactref element="DPC" pad="15"/>
+<contactref element="DPC" pad="16"/>
 <wire x1="26.8986" y1="9.4535" x2="26.8986" y2="8.6106" width="0.6096" layer="1"/>
 <wire x1="26.8986" y1="8.6106" x2="26.67" y2="8.128" width="0.6096" layer="1"/>
@@
 <wire x1="14.859" y1="8.636" x2="15.494" y2="8.636" width="0.8128" layer="1"/>
 <wire x1="25.974" y1="11.242" x2="25.974" y2="11.364" width="0.6096" layer="1"/>
-<contactref element="PORT2" pad="12"/>
+<contactref element="DPC" pad="12"/>
 <wire x1="40.005" y1="11.43" x2="37.846" y2="11.43" width="0.6096" layer="16"/>
 <wire x1="37.846" y1="11.43" x2="37.592" y2="11.176" width="0.6096" layer="16"/>
@@
 <wire x1="8.128" y1="8.928" x2="8.128" y2="8.89" width="0.6096" layer="1"/>
 <wire x1="5.588" y1="10.16" x2="5.588" y2="20.32" width="0.6096" layer="16"/>
-<contactref element="PORT2" pad="11"/>
+<contactref element="DPC" pad="11"/>
 <wire x1="42.545" y1="11.43" x2="42.545" y2="11.557" width="0.3048" layer="1"/>
 <wire x1="42.545" y1="11.557" x2="41.402" y2="12.7" width="0.3048" layer="1"/>
@@
 <signal name="TXDEN_1">
 <contactref element="U1" pad="22"/>
-<contactref element="PORT2" pad="1"/>
+<contactref element="DPC" pad="1"/>
 <wire x1="42.545" y1="24.13" x2="41.275" y2="22.86" width="0.254" layer="16"/>
 <wire x1="41.275" y1="22.86" x2="41.275" y2="5.461" width="0.254" layer="16"/>
@@
 <wire x1="28.194" y1="24.384" x2="29.464" y2="24.384" width="0.254" layer="16"/>
 <wire x1="30.734" y1="23.622" x2="30.226" y2="23.622" width="0.254" layer="1"/>
-<contactref element="PORT2" pad="10"/>
+<contactref element="DPC" pad="10"/>
 <wire x1="31.75" y1="14.478" x2="39.497" y2="14.478" width="0.254" layer="16"/>
 <wire x1="39.497" y1="14.478" x2="40.005" y2="13.97" width="0.254" layer="16"/>
@@
 <wire x1="28.956" y1="22.86" x2="28.956" y2="21.59" width="0.254" layer="1"/>
 <wire x1="28.956" y1="21.59" x2="29.718" y2="20.828" width="0.254" layer="1"/>
-<contactref element="PORT2" pad="8"/>
+<contactref element="DPC" pad="8"/>
 <wire x1="29.718" y1="16.256" x2="39.751" y2="16.256" width="0.254" layer="16"/>
 <wire x1="39.751" y1="16.256" x2="40.005" y2="16.51" width="0.254" layer="16"/>
@@
 <wire x1="18.034" y1="19.05" x2="18.46" y2="19.05" width="0.254" layer="1"/>
 <wire x1="18.46" y1="19.05" x2="18.57" y2="19.16" width="0.254" layer="1"/>
-<contactref element="PORT2" pad="14"/>
+<contactref element="DPC" pad="14"/>
 <via x="34.036" y="9.398" extent="1-16" drill="0.3556"/>
 <wire x1="34.036" y1="9.398" x2="34.036" y2="12.446" width="0.254" layer="1"/>
@@
 <wire x1="25.654" y1="23.114" x2="27.686" y2="23.114" width="0.254" layer="16"/>
 <wire x1="27.686" y1="23.114" x2="28.194" y2="23.622" width="0.254" layer="16"/>
-<contactref element="PORT2" pad="4"/>
+<contactref element="DPC" pad="4"/>
 <wire x1="28.194" y1="23.622" x2="37.973" y2="23.622" width="0.254" layer="16"/>
 <wire x1="37.973" y1="23.622" x2="40.005" y2="21.59" width="0.254" layer="16"/>
@@
 <wire x1="22.098" y1="17.272" x2="22.352" y2="17.018" width="0.254" layer="16"/>
 <wire x1="22.352" y1="17.018" x2="37.973" y2="17.018" width="0.254" layer="16"/>
-<contactref element="PORT2" pad="6"/>
+<contactref element="DPC" pad="6"/>
 <wire x1="37.973" y1="17.018" x2="40.005" y2="19.05" width="0.254" layer="16"/>
 </signal>
@@
 <wire x1="17.526" y1="19.812" x2="16.51" y2="19.812" width="0.254" layer="16"/>
 <wire x1="16.51" y1="19.812" x2="15.748" y2="20.828" width="0.254" layer="16"/>
-<contactref element="PORT2" pad="2"/>
+<contactref element="DPC" pad="2"/>
 <wire x1="17.78" y1="20.32" x2="38.608" y2="20.32" width="0.254" layer="16"/>
 <via x="38.608" y="20.32" extent="1-16" drill="0.3556"/>
