File: TSOC_USBUART2/revisions/R5_1/TSOC_USBUART2_R5_1.sch (EAGLE design)
At the start: 41 parts, among them J1 JMP-3-1_2, J2 JMP-3-1_2, U1 CY7C65215-32-PROTO, U2 AP2112K-3.3V

Commit message: update R5
Parts:
- renumbered PORT2 to DPC
Changed lines of the file:
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@@
 <part name="U$4" library="thingSoC" deviceset="TSOC-PCB" device="-SINGLE" value="TSOC-PCB-SINGLE"/>
 <part name="U$7" library="thingSoC" deviceset="TSOC-LOGO" device="-SMALL"/>
-<part name="PORT2" library="PatternAgents-ProtoPads" deviceset="M08X2" device=""/>
+<part name="DPC" library="PatternAgents-ProtoPads" deviceset="M08X2" device=""/>
 <part name="FUSE" library="Seeed-Fuse-2016" deviceset="SMD-PPTC-500MA(1206)" device="" value="SMD1206R500SF"/>
 <part name="ESD" library="Seeed-Diode-2016" deviceset="SMD-DIODE-TVS-5V-225MW(SOT-23)" device="" value="5V-225MW"/>
@@
 <instance part="U$4" gate="G$1" x="231.14" y="-147.32"/>
 <instance part="U$7" gate="G$1" x="127" y="-45.72"/>
-<instance part="PORT2" gate="G$1" x="134.62" y="-71.12"/>
+<instance part="DPC" gate="G$1" x="134.62" y="-71.12"/>
 <instance part="FUSE" gate="G$1" x="373.38" y="134.62" smashed="yes">
 <attribute name="NAME" x="375.92" y="137.668" size="1.778" layer="95"/>
@@
 <segment>
 <label x="116.84" y="-78.74" size="1.27" layer="95" font="vector" ratio="10" rot="MR0" xref="yes"/>
-<pinref part="PORT2" gate="G$1" pin="15"/>
+<pinref part="DPC" gate="G$1" pin="15"/>
 <wire x1="127" y1="-78.74" x2="116.84" y2="-78.74" width="0.1524" layer="91"/>
 </segment>
@@
 <wire x1="142.24" y1="-78.74" x2="152.4" y2="-78.74" width="0.1524" layer="91"/>
 <label x="152.4" y="-78.74" size="1.27" layer="95" font="vector" ratio="10" rot="MR180" xref="yes"/>
-<pinref part="PORT2" gate="G$1" pin="16"/>
+<pinref part="DPC" gate="G$1" pin="16"/>
 </segment>
 </net>
@@
 <wire x1="142.24" y1="-73.66" x2="152.4" y2="-73.66" width="0.1524" layer="91"/>
 <label x="152.4" y="-73.66" size="1.27" layer="95" font="vector" ratio="10" rot="MR180" xref="yes"/>
-<pinref part="PORT2" gate="G$1" pin="12"/>
+<pinref part="DPC" gate="G$1" pin="12"/>
 </segment>
 </net>
@@
 </segment>
 <segment>
-<pinref part="PORT2" gate="G$1" pin="1"/>
+<pinref part="DPC" gate="G$1" pin="1"/>
 <wire x1="127" y1="-60.96" x2="116.84" y2="-60.96" width="0.1524" layer="91"/>
 <label x="116.84" y="-60.96" size="1.27" layer="95" font="vector" ratio="10" rot="R180" xref="yes"/>
@@
 <wire x1="127" y1="-73.66" x2="116.84" y2="-73.66" width="0.1524" layer="91"/>
 <label x="116.84" y="-73.66" size="1.27" layer="95" font="vector" ratio="10" rot="MR0" xref="yes"/>
-<pinref part="PORT2" gate="G$1" pin="11"/>
+<pinref part="DPC" gate="G$1" pin="11"/>
 </segment>
 </net>
@@
 <wire x1="142.24" y1="-71.12" x2="152.4" y2="-71.12" width="0.1524" layer="91"/>
 <label x="152.4" y="-71.12" size="1.27" layer="95" font="vector" ratio="10" rot="MR180" xref="yes"/>
-<pinref part="PORT2" gate="G$1" pin="10"/>
+<pinref part="DPC" gate="G$1" pin="10"/>
 </segment>
 </net>
@@
 <wire x1="142.24" y1="-68.58" x2="152.4" y2="-68.58" width="0.1524" layer="91"/>
 <label x="152.4" y="-68.58" size="1.27" layer="95" font="vector" ratio="10" rot="MR180" xref="yes"/>
-<pinref part="PORT2" gate="G$1" pin="8"/>
+<pinref part="DPC" gate="G$1" pin="8"/>
 </segment>
 </net>
@@
 <wire x1="142.24" y1="-76.2" x2="152.4" y2="-76.2" width="0.1524" layer="91"/>
 <label x="152.4" y="-76.2" size="1.27" layer="95" font="vector" ratio="10" rot="MR180" xref="yes"/>
-<pinref part="PORT2" gate="G$1" pin="14"/>
+<pinref part="DPC" gate="G$1" pin="14"/>
 </segment>
 </net>
@@
 <wire x1="142.24" y1="-63.5" x2="152.4" y2="-63.5" width="0.1524" layer="91"/>
 <label x="152.4" y="-63.5" size="1.27" layer="95" font="vector" ratio="10" rot="MR180" xref="yes"/>
-<pinref part="PORT2" gate="G$1" pin="4"/>
+<pinref part="DPC" gate="G$1" pin="4"/>
 </segment>
 </net>
@@
 <wire x1="142.24" y1="-66.04" x2="152.4" y2="-66.04" width="0.1524" layer="91"/>
 <label x="152.4" y="-66.04" size="1.27" layer="95" font="vector" ratio="10" rot="MR180" xref="yes"/>
-<pinref part="PORT2" gate="G$1" pin="6"/>
+<pinref part="DPC" gate="G$1" pin="6"/>
 </segment>
 </net>
@@
 <wire x1="142.24" y1="-60.96" x2="152.4" y2="-60.96" width="0.1524" layer="91"/>
 <label x="152.4" y="-60.96" size="1.27" layer="95" font="vector" ratio="10" rot="MR180" xref="yes"/>
-<pinref part="PORT2" gate="G$1" pin="2"/>
-</segment>
-</net>
+<pinref part="DPC" gate="G$1" pin="2"/>
+</segment>
+</net>
